Commit message: fixed the intialize.m file to compile everything correctly and adjusted uarmtd_planner.m so kinova_grasp_simple_example.m works correctly with the mex code. also created some visualization files to create a blender video from a matlab simulation trial.

File: urdfs/kinova/Kinova_Grasp_Cylinder_Edge.urdf (robot description, URDF)
Before this commit: robot gen3_robotiq_2f_85, 11 links, 10 joints
Links:
- link base: geometry collision mesh filename=meshes/base_link.obj; visual mesh filename=meshes/base_link.obj
- link bracelet_link: geometry collision mesh filename=meshes/bracelet_with_vision_link.obj; visual mesh filename=meshes/bracelet_with_vision_link.obj
- link cube_link: geometry collision mesh filename=meshes/RTDForceCylinder_OriginShiftedScaled.obj; visual mesh filename=meshes/RTDForceCylinder_OriginShiftedScaled.obj
- link forearm_link: geometry collision mesh filename=meshes/forearm_link.obj; visual mesh filename=meshes/forearm_link.obj
- link gripper_base: geometry collision mesh filename=meshes/base_of_gripper.obj; visual mesh filename=meshes/base_of_gripper.obj
- link half_arm_1_link: geometry collision mesh filename=meshes/half_arm_1_link.obj; visual mesh filename=meshes/half_arm_1_link.obj
- link half_arm_2_link: geometry collision mesh filename=meshes/half_arm_2_link.obj; visual mesh filename=meshes/half_arm_2_link.obj
- link shoulder_link: geometry collision mesh filename=meshes/shoulder_link.obj; visual mesh filename=meshes/shoulder_link.obj
- link spherical_wrist_1_link: geometry collision mesh filename=meshes/spherical_wrist_1_link.obj; visual mesh filename=meshes/spherical_wrist_1_link.obj
- link spherical_wrist_2_link: geometry collision mesh filename=meshes/spherical_wrist_2_link.obj; visual mesh filename=meshes/spherical_wrist_2_link.obj
- link waiter_tray_link: geometry collision mesh filename=meshes/plate_shifted_scaled_origin_v3.obj; visual mesh filename=meshes/plate_shifted_scaled_origin_v3.obj

File: urdfs/kinova/Kinova_Grasp_w_Tray_Gripper.urdf (robot description, URDF)
Before this commit: robot gen3_robotiq_2f_85, 21 links, 20 joints
Links:
- link gripper_left_coupler: geometry collision mesh filename=meshes/left_coupler.STL; visual mesh filename=meshes/left_coupler.STL
- link gripper_left_driver: geometry collision mesh filename=meshes/left_driver.STL; visual mesh filename=meshes/left_driver.STL
- link gripper_left_follower: geometry collision mesh filename=meshes/left_follower.STL; visual mesh filename=meshes/left_follower.STL
- link gripper_left_pad: geometry collision mesh filename=meshes/left_pad.STL; visual mesh filename=meshes/left_pad.STL
- link gripper_left_spring_link: geometry collision mesh filename=meshes/left_spring_link.STL; visual mesh filename=meshes/left_spring_link.STL
- link gripper_right_coupler: geometry collision mesh filename=meshes/right_coupler.STL; visual mesh filename=meshes/right_coupler.STL
- link gripper_right_driver: geometry collision mesh filename=meshes/right_driver.STL; visual mesh filename=meshes/right_driver.STL
- link gripper_right_follower: geometry collision mesh filename=meshes/right_follower.STL; visual mesh filename=meshes/right_follower.STL
- link gripper_right_pad: geometry collision mesh filename=meshes/right_pad.STL; visual mesh filename=meshes/right_pad.STL
- link gripper_right_spring_link: geometry collision mesh filename=meshes/right_spring_link.STL; visual mesh filename=meshes/right_spring_link.STL
